Commit message: update world and fix controller

File: src/nautilus_description/urdf/gazebo.xacro (robot description, xacro)
@@ -10,4 +10,6 @@
     <xacro:property name="nautilus_width"  value="0.2286"/>
     <xacro:property name="nautilus_height" value="0.254"/>
+    <xacro:property name="cameraSize" value="0.1"/>
+    <xacro:property name="cameraMass" value="0.1"/>
     <xacro:macro name="nautilus_hydro_model" params="namespace">
       <!-- List of hydrodynamic models this robot's links -->

File: src/nautilus_description/urdf/sensors.xacro (robot description, xacro)
@@ -89,31 +89,3 @@
     </sensor>
   </gazebo>
-  <!-- Mount a GPS. -->
-  <xacro:default_gps namespace="${namespace}" parent_link="${namespace}/base_link" />
-  <!-- Mount a Pose 3D sensor. -->
-  <xacro:default_pose_3d namespace="${namespace}" parent_link="${namespace}/base_link" />
-  <!-- Forward-looking sonar sensor -->
-  <xacro:forward_multibeam_p900 namespace="${namespace}" parent_link="${namespace}/base_link">
-    <origin xyz="0 0 0" rpy="0 0 0"/>
-  </xacro:forward_multibeam_p900>
-  <!-- DVL  -->
-  <xacro:default_dvl namespace="${namespace}" parent_link="${namespace}/base_link">
-    <origin xyz="0 0 0" rpy="0 0 0"/>
-  </xacro:default_dvl>
-  <!-- RPT  -->
-  <xacro:default_rpt namespace="${namespace}" parent_link="${namespace}/base_link">
-    <origin xyz="0 0 0" rpy="0 0 0"/>
-  </xacro:default_rpt>
-  <!-- Pressure  -->
-  <xacro:default_pressure namespace="${namespace}" parent_link="${namespace}/base_link">
-    <origin xyz="0 0 0" rpy="0 0 0"/>
-  </xacro:default_pressure>
-  <!-- IMU  -->
-  <xacro:default_imu namespace="${namespace}" parent_link="${namespace}/base_link">
-    <origin xyz="0 0 0" rpy="0 0 0"/>
-  </xacro:default_imu>
-  <!-- Mount a camera  -->
-  <xacro:default_camera namespace="${namespace}" parent_link="${namespace}/base_link" suffix="">
-    <origin xyz="0 0 0" rpy="0 0 0"/>
-  </xacro:default_camera>
 </robot>

File: src/nautilus_description/urdf/snippets.xacro (robot description, xacro)
@@ -55,6 +55,6 @@
         <clampMin>-100</clampMin>
         <!-- Minimum and maximum thrust force output allowed -->
-        <thrustMin>-2.36</thrustMin>
-        <thrustMax>2.36</thrustMax>
+        <thrustMin>-10</thrustMin>
+        <thrustMax>10</thrustMax>
         <!--
         Value from 0 to 1 to set the efficiency of the output thrust force

Commit message: tune camera size

File: src/nautilus_description/urdf/gazebo.xacro (robot description, xacro)
@@ -10,6 +10,6 @@
     <xacro:property name="nautilus_width"  value="0.2286"/>
     <xacro:property name="nautilus_height" value="0.254"/>
-    <xacro:property name="cameraSize" value="0.1"/>
-    <xacro:property name="cameraMass" value="0.1"/>
+    <xacro:property name="cameraSize" value="0.01"/>
+    <xacro:property name="cameraMass" value="0.01"/>
     <xacro:macro name="nautilus_hydro_model" params="namespace">
       <!-- List of hydrodynamic models this robot's links -->
