Commit message: simulator has basic functionality

File: src/nautilus_description/urdf/base.xacro (robot description, xacro)
@@ -39,7 +39,7 @@
           <mass value="${mass}" />
           <origin xyz="${cog}" rpy="0 0 0"/>
-          <inertia ixx="525.39" ixy="1.44" ixz="33.41"
-                   iyy="794.20" iyz="2.6"
-                   izz="691.23" />
+          <inertia ixx="300" ixy="1" ixz="30"
+                   iyy="400" iyz="2"
+                   izz="500" />
         </inertial>
         <visual>

File: src/nautilus_description/urdf/snippets.xacro (robot description, xacro)
@@ -7,5 +7,5 @@
   over propeller's frame X-axis in DAE (Collada) or STL format.
   -->
-  <xacro:property name="prop_mesh_file" value="file://$(find nautilus_description)/meshes/propeller.dae"/>
+  <xacro:property name="prop_mesh_file" value="file://$(find nautilus_description)/meshes/t100.dae"/>
   <!--
     Thruster macro with integration of joint and link. The thrusters should
@@ -53,7 +53,7 @@
         <clampMax>100</clampMax>
         <!-- Minimum allowed value for the input signal for thruster unit -->
-        <clampMin>0</clampMin>
+        <clampMin>-100</clampMin>
         <!-- Minimum and maximum thrust force output allowed -->
-        <thrustMin>-1.5</thrustMin>
+        <thrustMin>-2.36</thrustMin>
         <thrustMax>2.36</thrustMax>
         <!--

Commit message: added camera

File: src/nautilus_description/urdf/base.xacro (robot description, xacro)
@@ -78,5 +78,5 @@
     <xacro:include filename="$(find nautilus_description)/urdf/actuators.xacro"/>
     <!-- Include the sensor modules -->
-    <!-- <xacro:include filename="$(find nautilus_description)/urdf/sensors.xacro"/> -->
+    <xacro:include filename="$(find nautilus_description)/urdf/sensors.xacro"/>
   </xacro:macro>
 </robot>

File: src/nautilus_description/urdf/sensors.xacro (robot description, xacro)
@@ -7,4 +7,86 @@
     more examples or add you own custom sensor units.
   -->
+  <!-- adding camera link -->
+  <link name="camera_link">
+    <!-- collision properties -->
+    <collision>
+      <origin xyz="0 0 0" rpy="0 0 0"/>
+      <geometry>
+        <box size="${cameraSize} ${cameraSize} ${cameraSize}"/>
+      </geometry>
+    </collision>
+    <!-- visual properties -->
+    <visual>
+      <origin xyz="0 0 0" rpy="0 0 0"/>
+      <geometry>
+        <box size="${cameraSize} ${cameraSize} ${cameraSize}"/>
+      </geometry>
+      <material name="green"/>
+    </visual>
+   <!-- inertial properties -->
+    <inertial>
+      <mass value="${cameraMass}" />
+      <origin xyz="0 0 0" rpy="0 0 0"/>
+      <box_inertia m="${cameraMass}" x="${cameraSize}" y="${cameraSize}" z="${cameraSize}" />
+      <inertia ixx="1e-6" ixy="0" ixz="0" iyy="1e-6" iyz="0" izz="1e-6" />
+    </inertial>
+  </link>
+  <!-- Adding camera joint -->
+  <joint name="camera_joint" type="fixed">
+    <axis xyz="0 1 0" />
+    <!-- position relative to the parent link -->
+    <origin xyz="0.21 0 0" rpy="0 0 0"/>
+    <parent link="nautilus/base_link"/>
+    <child link="camera_link"/>
+  </joint>
+  <!-- Adding gazebo plugins -->>
+  <gazebo reference="camera_link">
+    <!-- Defining camera properties -->
+    <sensor type="camera" name="camera1">
+      <update_rate>30.0</update_rate>
+      <camera name="head">
+        <horizontal_fov>1.3962634</horizontal_fov>
+        <image>
+          <width>800</width>
+          <height>800</height>
+          <format>R8G8B8</format>
+        </image>
+        <clip>
+          <near>0.02</near>
+          <far>300</far>
+        </clip>
+        <noise>
+          <type>gaussian</type>
+          <!-- Noise is sampled independently per pixel on each frame.
+               That pixel's noise value is added to each of its color
+               channels, which at that point lie in the range [0,1]. -->
+          <mean>0.0</mean>
+          <stddev>0.007</stddev>
+        </noise>
+      </camera>
+      <plugin name="camera_controller" filename="libgazebo_ros_camera.so">
+        <alwaysOn>true</alwaysOn>
+        <updateRate>0.0</updateRate>
+        <!-- rostopic name: nautilus/camera1/nautilus_cam -->
+        <cameraName>nautilus/camera1</cameraName>
+        <imageTopicName>nautilus_cam</imageTopicName>
+        <cameraInfoTopicName>camera_info</cameraInfoTopicName>
+        <frameName>camera_link_optical</frameName>
+        <!-- setting hackBaseline to anything but 0.0 will cause a misalignment
+            between the gazebo sensor image and the frame it is supposed to
+            be attached to -->
+        <hackBaseline>0.0</hackBaseline>
+        <distortionK1>0.0</distortionK1>
+        <distortionK2>0.0</distortionK2>
+        <distortionK3>0.0</distortionK3>
+        <distortionT1>0.0</distortionT1>
+        <distortionT2>0.0</distortionT2>
+        <CxPrime>0</CxPrime>
+        <Cx>0.0</Cx>
+        <Cy>0.0</Cy>
+        <focalLength>0.0</focalLength>
+      </plugin>
+    </sensor>
+  </gazebo>
   <!-- Mount a GPS. -->
   <xacro:default_gps namespace="${namespace}" parent_link="${namespace}/base_link" />

Commit message: fix typos, add wall to colony_dead_bleach.dae

File: src/nautilus_description/urdf/base.xacro (robot description, xacro)
@@ -52,5 +52,5 @@
         <origin xyz="0 0 -0.75" rpy="0 0 0"/>
         <geometry>
-          <box size="2.56 1.50 0.10"/>
+          <box size="0.01 0.01 0.01"/>
         </geometry>
       </collision>
@@ -58,14 +58,14 @@
       <collision>
         <origin xyz="0 0 0.60" rpy="0 0 0"/>
-        <geometry><box size="0.381 0.2286 0.1"/></geometry>
+        <geometry><box size="0.01 0.01 0.01"/></geometry>
       </collision>
       <!-- left / right sides -->
       <collision>
         <origin xyz="-0.20 0.70 -0.15" rpy="0 0 0"/>
-        <geometry><box size="0.381 0.1 0.254"/></geometry>
+        <geometry><box size="0.01 0.01 0.01"/></geometry>
       </collision>
       <collision>
         <origin xyz="-0.20 -0.70 -0.15" rpy="0 0 0"/>
-        <geometry><box size="0.381 0.1 0.254"/></geometry>
+        <geometry><box size="0.01 0.01 0.01"/></geometry>
       </collision>
       </link>

File: src/nautilus_description/urdf/gazebo.xacro (robot description, xacro)
@@ -10,6 +10,6 @@
     <xacro:property name="nautilus_width"  value="0.2286"/>
     <xacro:property name="nautilus_height" value="0.254"/>
-    <xacro:property name="cameraSize" value="0.01"/>
-    <xacro:property name="cameraMass" value="0.01"/>
+    <xacro:property name="cameraSize" value="0.1"/>
+    <xacro:property name="cameraMass" value="0.1"/>
     <xacro:macro name="nautilus_hydro_model" params="namespace">
       <!-- List of hydrodynamic models this robot's links -->
